Commit message: Wheel-leg roll guard, room-based task split, localhost DDS profile, README for wheel-leg robot

File: src/rescue_description/urdf/wheelleg.urdf.xacro (robot description, xacro)
@@ -16,5 +16,5 @@
   and the legs can't move), applies the differential and levels the body from its roll.
   base_link is the body centre, ~0.49 m above the ground at the default 0.5 rad stance.
-  Skid steering only turns while the wheelbase is no longer than the track (0.48 m):
+  Skid steering only turns while the wheelbase is no longer than the track (0.44 m):
   above ~0.65 rad (wide stance) it drives straight but can't turn on the spot.
 -->
@@ -27,10 +27,10 @@
   <xacro:property name="body_w" value="0.30"/>
   <xacro:property name="body_h" value="0.12"/>
-  <xacro:property name="hub_y" value="0.18"/>
+  <xacro:property name="hub_y" value="0.165"/>
   <xacro:property name="hub_z" value="-0.04"/>
   <xacro:property name="leg_l" value="0.36"/>
   <xacro:property name="wheel_r" value="0.14"/>
   <xacro:property name="wheel_w" value="0.08"/>
-  <xacro:property name="wheel_y" value="0.06"/>         <!-- wheel centre outboard of its leg -->
+  <xacro:property name="wheel_y" value="0.055"/>        <!-- wheel centre outboard of its leg: track 0.44, width 0.52 -->
   <material name="red"><color rgba="0.86 0.06 0.05 1"/></material>
   <material name="dark"><color rgba="0.08 0.08 0.09 1"/></material>
@@ -179,7 +179,13 @@
       <leg_max_rate>1.2</leg_max_rate>
       <diff_gain>8.0</diff_gain>
-      <rocker_free>0.15</rocker_free>
-      <rocker_turn>0.12</rocker_turn>
-      <level_gain>1.5</level_gain>
+      <climb_open>0.2</climb_open>
+      <climb_close>0.3</climb_close>
+      <climb_rate>0.5</climb_rate>
+      <push_time>1.5</push_time>
+      <stall_time>0.4</stall_time>
+      <climb_attempts>0</climb_attempts>   <!-- leg pushes off: tested, they tip the robot at the turnable stance -->
+      <tip_pitch>0.35</tip_pitch>
+      <roll_guard>0.2</roll_guard>
+      <level_gain>3.0</level_gain>
       <level_limit>0.4</level_limit>
       <max_speed>0.9</max_speed>

Commit message: Wheel-leg: wider stance, wall guard, centred paths, home-return and controller fixes; swarm: robot health and takeover of a fallen robot's rooms

File: src/rescue_description/urdf/wheelleg.urdf.xacro (robot description, xacro)
@@ -15,12 +15,12 @@
   It also turns the wheels to match the legs' motion (otherwise the tyres pin the feet
   and the legs can't move), applies the differential and levels the body from its roll.
-  base_link is the body centre, ~0.49 m above the ground at the default 0.5 rad stance.
-  Skid steering only turns while the wheelbase is no longer than the track (0.44 m):
-  above ~0.65 rad (wide stance) it drives straight but can't turn on the spot.
+  base_link is the body centre, ~0.43 m above the ground at the default 0.8 rad stance
+  (wheelbase 0.52 m). Skid steering only turns while the wheelbase is no longer than the
+  track (0.52 m): much above 0.8 rad it drives straight but can't turn on the spot.
 -->
 <robot name="wheelleg" xmlns:xacro="http://www.ros.org/wiki/xacro">
   <xacro:arg name="ns" default="r1"/>
   <xacro:arg name="sensors" default="true"/>
-  <xacro:arg name="stance" default="0.5"/>
+  <xacro:arg name="stance" default="0.8"/>
   <xacro:property name="ns" value="$(arg ns)"/>
   <xacro:property name="body_l" value="0.54"/>         <!-- straight section; ends are rounded -->
@@ -32,5 +32,5 @@
   <xacro:property name="wheel_r" value="0.14"/>
   <xacro:property name="wheel_w" value="0.08"/>
-  <xacro:property name="wheel_y" value="0.055"/>        <!-- wheel centre outboard of its leg: track 0.44, width 0.52 -->
+  <xacro:property name="wheel_y" value="0.095"/>        <!-- wheel centre outboard of its leg: track 0.52, width 0.60 -->
   <material name="red"><color rgba="0.86 0.06 0.05 1"/></material>
   <material name="dark"><color rgba="0.08 0.08 0.09 1"/></material>
@@ -172,5 +172,5 @@
       <leg_length>${leg_l}</leg_length>
       <wheel_radius>${wheel_r}</wheel_radius>
-      <track>${2*(hub_y + wheel_y)}</track>
+      <track>${2*(hub_y + wheel_y) * 1.8}</track>   <!-- x1.8: tyres scrub turning on the spot (measured) -->
       <stance>$(arg stance)</stance>
       <stance_min>0.25</stance_min>
